File: hardware/dashboard-plusplus-carrier.kicad_pcb (KiCad board)
At the start: 4 copper layers, 95 x 55 mm, 56 parts, among them J1 XT30U-M, J10a ESP32-DEVKIT-A, J10b ESP32-DEVKIT-B, J13 DEBUG, J14 TRIP + EN, J15 SPARE, J16 SPARE N, J17 IGN + COOLANT, J18 SPARE S, J3 TFT-ILI9488, J6 LDR + FUEL, J8 GPS_PADS, J9 HALL, Q1 IRFR9540N, U4 DPP_DCDC_MODULE

Commit message: Name every JST-PH pad with standing silks, drop pair captions
Other:
- board text added: "+V"
- board text added: "G"
- board text added: "J6 LDR GND FUEL GND J9 +V SIG G"
- board text added: "SIG"
- board text removed: "J6 LDR GND FUEL GND J9 +V SIG GND"
Changed lines of the file:
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@@
 (gr_text "OUT+" (at 116.45 128.74 0.0) (layer "B.SilkS") (effects (font (size 0.90 0.90) (thickness 0.12)) (justify left top mirror)))
 (gr_text "OUT-" (at 133.45 128.74 0.0) (layer "B.SilkS") (effects (font (size 0.90 0.90) (thickness 0.12)) (justify left top mirror)))
-(gr_text "TRIP" (at 166.30 88.50 0.0) (layer "B.SilkS") (effects (font (size 0.80 0.80) (thickness 0.12)) (justify left top mirror)))
-(gr_text "EN" (at 169.78 88.50 0.0) (layer "B.SilkS") (effects (font (size 0.80 0.80) (thickness 0.12)) (justify left top mirror)))
-(gr_text "IGN" (at 180.41 88.50 0.0) (layer "B.SilkS") (effects (font (size 0.80 0.80) (thickness 0.12)) (justify left top mirror)))
-(gr_text "COOL" (at 184.96 88.50 0.0) (layer "B.SilkS") (effects (font (size 0.80 0.80) (thickness 0.12)) (justify left top mirror)))
-(gr_text "LDR" (at 186.53 120.40 0.0) (layer "B.SilkS") (effects (font (size 0.80 0.80) (thickness 0.12)) (justify left top mirror)))
-(gr_text "FUEL" (at 182.84 120.40 0.0) (layer "B.SilkS") (effects (font (size 0.80 0.80) (thickness 0.12)) (justify left top mirror)))
-(gr_text "HALL" (at 169.41 120.40 0.0) (layer "B.SilkS") (effects (font (size 0.80 0.80) (thickness 0.12)) (justify left top mirror)))
+(gr_text "IGN" (at 179.40 89.52 270.0) (layer "B.SilkS") (effects (font (size 0.80 0.80) (thickness 0.12)) (justify mirror)))
+(gr_text "GND" (at 181.40 89.52 270.0) (layer "B.SilkS") (effects (font (size 0.80 0.80) (thickness 0.12)) (justify mirror)))
+(gr_text "COOL" (at 183.40 89.52 270.0) (layer "B.SilkS") (effects (font (size 0.80 0.80) (thickness 0.12)) (justify mirror)))
+(gr_text "GND" (at 185.40 89.52 270.0) (layer "B.SilkS") (effects (font (size 0.80 0.80) (thickness 0.12)) (justify mirror)))
+(gr_text "TRIP" (at 165.00 89.52 270.0) (layer "B.SilkS") (effects (font (size 0.80 0.80) (thickness 0.12)) (justify mirror)))
+(gr_text "GND" (at 167.00 89.52 270.0) (layer "B.SilkS") (effects (font (size 0.80 0.80) (thickness 0.12)) (justify mirror)))
+(gr_text "EN" (at 169.00 89.52 270.0) (layer "B.SilkS") (effects (font (size 0.80 0.80) (thickness 0.12)) (justify mirror)))
+(gr_text "GND" (at 171.00 89.52 270.0) (layer "B.SilkS") (effects (font (size 0.80 0.80) (thickness 0.12)) (justify mirror)))
+(gr_text "LDR" (at 185.40 120.48 270.0) (layer "B.SilkS") (effects (font (size 0.80 0.80) (thickness 0.12)) (justify mirror)))
+(gr_text "GND" (at 183.40 120.48 270.0) (layer "B.SilkS") (effects (font (size 0.80 0.80) (thickness 0.12)) (justify mirror)))
+(gr_text "FUEL" (at 181.40 120.48 270.0) (layer "B.SilkS") (effects (font (size 0.80 0.80) (thickness 0.12)) (justify mirror)))
+(gr_text "GND" (at 179.40 120.48 270.0) (layer "B.SilkS") (effects (font (size 0.80 0.80) (thickness 0.12)) (justify mirror)))
+(gr_text "+V" (at 170.00 120.48 270.0) (layer "B.SilkS") (effects (font (size 0.80 0.80) (thickness 0.12)) (justify mirror)))
+(gr_text "SIG" (at 168.00 120.48 270.0) (layer "B.SilkS") (effects (font (size 0.80 0.80) (thickness 0.12)) (justify mirror)))
+(gr_text "G" (at 166.00 120.48 270.0) (layer "B.SilkS") (effects (font (size 0.80 0.80) (thickness 0.12)) (justify mirror)))
 (gr_text "GNSS" (at 160.00 80.40 0.0) (layer "B.SilkS") (effects (font (size 0.80 0.80) (thickness 0.12)) (justify left top mirror)))
 (gr_text "IGN" (at 152.06 79.24 0.0) (layer "F.SilkS") (effects (font (size 0.80 0.80) (thickness 0.12)) (justify left top)))
@@
 (gr_text "  19 21 3 1 22 23" (at 111.50 146.90 0.0) (layer "Dwgs.User") (effects (font (size 1.00 1.00) (thickness 0.12)) (justify left top)))
 (gr_text "J17 IGN GND COOL GND   J14 TRIP GND EN GND" (at 111.50 148.40 0.0) (layer "Dwgs.User") (effects (font (size 1.00 1.00) (thickness 0.12)) (justify left top)))
-(gr_text "J6 LDR GND FUEL GND    J9 +V SIG GND" (at 111.50 149.90 0.0) (layer "Dwgs.User") (effects (font (size 1.00 1.00) (thickness 0.12)) (justify left top)))
+(gr_text "J6 LDR GND FUEL GND    J9 +V SIG G" (at 111.50 149.90 0.0) (layer "Dwgs.User") (effects (font (size 1.00 1.00) (thickness 0.12)) (justify left top)))
 (gr_text "JST = right-angle SMD, bodies under the board; pin 1 is at the" (at 111.50 151.40 0.0) (layer "Dwgs.User") (effects (font (size 1.00 1.00) (thickness 0.12)) (justify left top)))
 (gr_text "west end of the north pair, east end of the south pair (top view)" (at 111.50 152.90 0.0) (layer "Dwgs.User") (effects (font (size 1.00 1.00) (thickness 0.12)) (justify left top)))
